File: tests/test_dr.kicad_pcb (KiCad board)
At the start: 2 copper layers, 4 parts

Commit message: Moved from using @staticmethod to a more object oriented approach so specialized data/flags could be placed in the objects to affect operations. * Added inject/eject for board design rules (not fully working).
Other:
- rule trace_min: 0.2 -> 0.012345
- rule via_min_drill: 0.3 -> 0.056789
- rule via_min_size: 0.2 -> 0.078901
Changed lines of the file:
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@@
 (kicad_pcb (version 20171130) (host pcbnew "(5.1.2)-1")
   (general
-    (thickness 1.6)
+    (thickness 0.034567)
     (drawings 0)
     (tracks 0)
@@
   (setup
     (last_trace_width 0.25)
+    (user_trace_width 0.65)
     (user_trace_width 1)
-    (user_trace_width 0.65)
     (trace_clearance 0.2)
     (zone_clearance 0.508)
     (zone_45_only no)
-    (trace_min 0.2)
+    (trace_min 0.012345)
     (via_size 0.8)
     (via_drill 0.4)
-    (via_min_size 0.2)
-    (via_min_drill 0.3)
+    (via_min_size 0.078901)
+    (via_min_drill 0.056789)
+    (blind_buried_vias_allowed yes)
     (uvia_size 0.3)
     (uvia_drill 0.1)
     (uvias_allowed no)
-    (uvia_min_size 0.2)
-    (uvia_min_drill 0.1)
+    (uvia_min_size 0.06789)
+    (uvia_min_drill 0.045678)
     (edge_width 0.05)
     (segment_width 0.2)
